File: lv_amp.kicad_sch (KiCad schematic)
At the start: 87 parts

Commit message: power supply parts
Parts:
- added TP9: TestPoint, symbol Connector:TestPoint
- C11, C14: renamed from C?; footprint (none) -> Capacitor_SMD:C_0805_2012Metric
- C13: renamed from C?; footprint (none) -> Capacitor_Tantalum_SMD:CP_EIA-6032-28_Kemet-C
- C15: renamed from C?; value 1uF -> 0.1uF; footprint (none) -> Capacitor_SMD:C_0805_2012Metric
- C17: renamed from C?; footprint (none) -> Capacitor_Tantalum_SMD:CP_EIA-7343-43_Kemet-X
- C20: renamed from C?; footprint (none) -> Capacitor_SMD:CP_Elec_10x10
- C22: renamed from C?; footprint (none) -> Capacitor_SMD:CP_Elec_16x17.5
- D1: renamed from D?; footprint (none) -> Package_TO_SOT_SMD:TO-263-2_TabPin1
- L1: renamed from L?; value L -> 56uH; footprint (none) -> lv_amp:pm2110
- Q1: renamed from Q?; footprint (none) -> Package_TO_SOT_SMD:TO-263-2; symbol Device:Q_NMOS_DGS -> Device:Q_NMOS_GDS
- R21: renamed from R?; value R_US -> 0.100; footprint (none) -> Resistor_SMD:R_2512_6332Metric
- R24: renamed from R?; value R_US -> 2Meg; footprint (none) -> Resistor_SMD:R_2512_6332Metric
- R25: renamed from R?; value R_US -> 10k; footprint (none) -> Resistor_SMD:R_0603_1608Metric
- gave numbers to parts that had none: 66
Connections:
- net GND: now also TP9.1
- net at D1.2 (A), L1.2: now also Q1.2 (D); no longer Q1.1 (D)
- net at U5.1 (EXT): now also Q1.1 (G); no longer Q1.2 (G)
Other:
- moved on the sheet: TP2, TP3, TP4

Commit message: WIP
Connections:
- net at RV2.3: now also C2.2, RV1.1
- net at C1.2: now also RV1.3; no longer RV1.1
- now unconnected: RV2.1
Other:
- moved on the sheet: RV2
Changed lines of the file:
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@@
     (pin "9")
   )
-  (symbol (lib_id "Device:R_Potentiometer_US") (at 43.18 168.91 90) (unit 1)
+  (symbol (lib_id "Device:R_Potentiometer_US") (at 43.18 168.91 270) (mirror x) (unit 1)
     (in_bom yes) (on_board yes) (fields_autoplaced)
     (property "Reference" "RV2" (id 0) (at 43.18 171.9485 90))
@@
     (pin "1")
   )
-  (symbol (lib_id "Device:R_Potentiometer_US") (at 36.83 160.02 0) (unit 1)
+  (symbol (lib_id "Device:R_Potentiometer_US") (at 36.83 160.02 0) (mirror x) (unit 1)
     (in_bom yes) (on_board yes)
-    (property "Reference" "RV1" (id 0) (at 40.64 156.21 0)
-      (effects (font (size 1.27 1.27)) (justify right))
-    )
-    (property "Value" "250k" (id 1) (at 43.18 162.56 0)
-      (effects (font (size 1.27 1.27)) (justify right))
-    )
+    (property "Reference" "RV1" (id 0) (at 40.64 163.83 0)
+      (effects (font (size 1.27 1.27)) (justify right))
+    )
+    (property "Value" "250k" (id 1) (at 43.18 157.48 0)
+      (effects (font (size 1.27 1.27)) (justify right))
+    )

Commit message: update footprints
Parts:
- R1, R12, R16, R2, R26, R3, R32, R33, R4, R5, R6, R9: footprint (none) -> Resistor_SMD:R_0603_1608Metric
- R10, R11, R14, R15, R23, R29, R8: footprint (none) -> Resistor_SMD:R_1206_3216Metric
- R13, R18, R27, R31: footprint (none) -> Resistor_SMD:R_2512_6332Metric
- R17: footprint (none) -> Resistor_SMD:R_0805_2012Metric
- R19, R20, R22, R28, R30, R7: footprint (none) -> Resistor_SMD:R_1210_3225Metric
- TP1, TP2, TP3, TP4, TP5, TP6, TP7, TP8, TP9: footprint (none) -> TestPoint:TestPoint_THTPad_2.0x2.0mm_Drill1.0mm
- U2: footprint (none) -> Package_SO:SO-8_3.9x4.9mm_P1.27mm
Connections:
- no-connect marks 0 -> 4

Commit message: caps
Parts:
- C1: footprint (none) -> Capacitor_SMD:C_0603_1608Metric
- C10, C19, C5: footprint (none) -> Capacitor_SMD:CP_Elec_4x5.4; symbol Device:C -> Device:C_Polarized_US
- C12, C18, C21, C6: value .02uF -> 0.022uF; footprint (none) -> Capacitor_THT:C_Rect_L13.0mm_W4.0mm_P10.00mm_FKS3_FKP3_MKS4
- C13, C20, C22: symbol Device:C_Polarized -> Device:C_Polarized_US
- C16: footprint (none) -> Capacitor_THT:C_Rect_L18.0mm_W5.0mm_P15.00mm_FKS3_FKP3
- C2, C3: value 0.02uF -> 0.022uF; footprint (none) -> Capacitor_SMD:C_0805_2012Metric
- C23: footprint (none) -> Capacitor_THT:C_Rect_L18.0mm_W7.0mm_P15.00mm_FKS3_FKP3
- C4, C9: value 0.56uF -> 1uF; footprint (none) -> Capacitor_THT:C_Rect_L18.0mm_W7.0mm_P15.00mm_FKS3_FKP3
- C7: value 2000pF -> 2200pF; footprint (none) -> Capacitor_SMD:C_0805_2012Metric
- C8: footprint (none) -> Capacitor_SMD:C_0805_2012Metric

Commit message: footprints
Parts:
- C1: value 470pF -> 220pF
- C17: symbol Device:C_Polarized -> Device:C_Polarized_US
- J1, J3: footprint (none) -> Connector_Audio:Jack_6.35mm_Neutrik_NRJ4HF_Horizontal; symbol Connector:AudioJack2 -> Connector:AudioJack2_Switch
- J2: footprint (none) -> lv_amp:Kobiconn 179PH; symbol Connector:Jack-DC -> Connector:Barrel_Jack_Switch
- RV1: value 250k -> 500k; footprint (none) -> Potentiometer_THT:Potentiometer_Piher_T-16H_Single_Horizontal; Source (none) -> https://www.tubesandmore.com/products/potentiometer-alpha-a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
- RV2: value 25k -> 1meg; footprint (none) -> Potentiometer_THT:Potentiometer_Piher_T-16H_Single_Horizontal; source (none) -> https://www.tubesandmore.com/products/potentiometer-alpha-a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
- RV3, RV4: footprint (none) -> Potentiometer_THT:Potentiometer_Piher_T-16H_Single_Horizontal; Source (none) -> https://www.tubesandmore.com/products/potentiometer-alpha-a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
- U1, U3, U4: footprint Valve:Valve_Noval_P -> lv_amp:12ax7
- U1, U3, U4: footprint Valve:Valve_Noval_P -> lv_amp:12ax7; Source (none) -> https://www.tubesandmore.com/products/socket-9-pin-ceramic-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
Connections:
- net GND: now also J1.SN, J1.TN, RV4.1; no longer RV4.3
- net at C7.2, C8.1, R10.2: now also RV4.3; no longer RV4.1
- net at RV2.1: now also C2.2, RV1.1
- now unconnected: RV2.3
- no-connect marks 4 -> 8
Other:
- note added: "bass"
- note added: "expect center negative 12v"
- note added: "mid"
- note added: "treble"
- moved on the sheet: RV2
